File: ESP_Writer_BRD_v1.0.0/ESPWriter.brd (EAGLE design)
At the start: 40 x 60 mm, 13 parts

Commit message: update board
Connections:
- net N$4: now also JP3.4; no longer JP3.6
- net N$5: now also JP3.6; no longer JP3.4
Routing:
- net N$4: track 55.2 -> 32.6 mm
- net N$3: track 34.8 -> 33.8 mm
- net N$5: track 34.6 -> 35.7 mm
Changed lines of the file:
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@@
 <setting verticaltext="up"/>
 </settings>
-<grid distance="1.27" unitdist="mm" unit="mm" style="dots" multiple="1" display="yes" altdistance="5" altunitdist="mil" altunit="mm"/>
+<grid distance="0.15" unitdist="mm" unit="mm" style="dots" multiple="1" display="yes" altdistance="5" altunitdist="mil" altunit="mm"/>
 <layers>
 <layer number="1" name="Top" color="4" fill="1" visible="yes" active="yes"/>
@@
 <layer number="151" name="HeatSink" color="7" fill="1" visible="no" active="yes"/>
 <layer number="199" name="Contour" color="7" fill="1" visible="no" active="yes"/>
-<layer number="200" name="200bmp" color="1" fill="10" visible="yes" active="yes"/>
+<layer number="200" name="200bmp" color="1" fill="10" visible="no" active="yes"/>
 <layer number="201" name="201bmp" color="2" fill="1" visible="no" active="no"/>
 <layer number="202" name="202bmp" color="3" fill="1" visible="no" active="no"/>
@@
 <text x="6.35" y="24.13" size="1.016" layer="25" align="center-left">RXD</text>
 <text x="6.35" y="19.05" size="1.016" layer="25" align="center-left">GND</text>
-<text x="32.7025" y="33.0835" size="0.6096" layer="25" rot="R180" align="center">RXD</text>
-<text x="30.7975" y="33.0835" size="0.6096" layer="25" rot="R180" align="center">TXD</text>
+<text x="32.7025" y="33.0835" size="0.6096" layer="25" rot="R180" align="center">TXD</text>
+<text x="30.7975" y="33.0835" size="0.6096" layer="25" rot="R180" align="center">RXD</text>
 <text x="28.8925" y="31.8135" size="0.6096" layer="25" rot="R180" align="center">3V3</text>
 <text x="28.8925" y="33.0835" size="0.6096" layer="25" rot="R180" align="center">GND</text>
@@
 /CREATE-ROCKET
 /Avi_ESP_Hardware_Utility</text>
+<wire x1="34.671" y1="33.02" x2="34.036" y2="33.655" width="0.0762" layer="21"/>
+<wire x1="34.671" y1="33.02" x2="35.179" y2="32.512" width="0.0762" layer="21"/>
 </plain>
 <attributes>
@@
 <wire x1="7.62" y1="33.02" x2="6.35" y2="31.75" width="0.508" layer="16"/>
 <wire x1="6.35" y1="31.75" x2="3.81" y2="31.75" width="0.508" layer="16"/>
-<wire x1="31.75" y1="27.94" x2="31.75" y2="32.131" width="0.508" layer="16"/>
-<wire x1="31.75" y1="32.131" x2="30.861" y2="33.02" width="0.508" layer="16"/>
-<wire x1="30.861" y1="33.02" x2="7.62" y2="33.02" width="0.508" layer="16"/>
+<wire x1="31.75" y1="27.94" x2="31.75" y2="30.331" width="0.508" layer="16"/>
+<wire x1="31.75" y1="30.331" x2="29.061" y2="33.02" width="0.508" layer="16"/>
+<wire x1="29.061" y1="33.02" x2="7.62" y2="33.02" width="0.508" layer="16"/>
 </signal>
 <signal name="N$4">
-<contactref element="JP3" pad="6"/>
 <contactref element="JP1" pad="5"/>
-<wire x1="33.02" y1="29.21" x2="33.02" y2="35.56" width="0.508" layer="1"/>
-<wire x1="1.27" y1="36.83" x2="1.27" y2="25.4" width="0.508" layer="1"/>
-<wire x1="1.27" y1="25.4" x2="2.54" y2="24.13" width="0.508" layer="1"/>
-<wire x1="2.54" y1="24.13" x2="3.81" y2="24.13" width="0.508" layer="1"/>
-<wire x1="33.02" y1="35.56" x2="29.21" y2="39.37" width="0.508" layer="1"/>
-<wire x1="29.21" y1="39.37" x2="3.81" y2="39.37" width="0.508" layer="1"/>
-<wire x1="3.81" y1="39.37" x2="1.27" y2="36.83" width="0.508" layer="1"/>
+<contactref element="JP3" pad="4"/>
+<wire x1="30.48" y1="29.21" x2="28.49" y2="31.2" width="0.508" layer="1"/>
+<wire x1="28.49" y1="31.2" x2="25.05" y2="31.2" width="0.508" layer="1"/>
+<wire x1="25.05" y1="31.2" x2="24.3" y2="30.45" width="0.508" layer="1"/>
+<wire x1="24.3" y1="30.45" x2="12" y2="30.45" width="0.508" layer="1"/>
+<wire x1="10.8" y1="29.25" x2="12" y2="30.45" width="0.508" layer="1"/>
+<wire x1="3.81" y1="24.13" x2="9.43" y2="24.13" width="0.508" layer="1"/>
+<wire x1="9.43" y1="24.13" x2="10.8" y2="25.5" width="0.508" layer="1"/>
+<wire x1="10.8" y1="25.5" x2="10.8" y2="29.25" width="0.508" layer="1"/>
 </signal>
 <signal name="N$5">
-<contactref element="JP3" pad="4"/>
 <contactref element="JP1" pad="1"/>
-<wire x1="30.48" y1="29.21" x2="30.48" y2="34.29" width="0.508" layer="1"/>
-<wire x1="30.48" y1="34.29" x2="27.94" y2="36.83" width="0.508" layer="1"/>
 <wire x1="5.08" y1="36.83" x2="3.81" y2="35.56" width="0.508" layer="1"/>
 <wire x1="3.81" y1="35.56" x2="3.81" y2="34.29" width="0.508" layer="1"/>
 <wire x1="27.94" y1="36.83" x2="5.08" y2="36.83" width="0.508" layer="1"/>
+<contactref element="JP3" pad="6"/>
+<wire x1="33.02" y1="29.21" x2="33.02" y2="31.75" width="0.508" layer="1"/>
+<wire x1="33.02" y1="31.75" x2="27.94" y2="36.83" width="0.508" layer="1"/>
 </signal>
 <signal name="N$6">
